File: pcb/bakeneko-65-pcb.kicad_pcb (KiCad board)
At the start: 2 copper layers, 303.8 x 94.2 mm, 161 parts, among them J1 JST SH 4-pin, J2 AVR-ISP-6, SW1 Reset, U1 SRV05-4, U2 ATmega32U4-AU, Y1 16MHz

Commit message: Modified PCB for hotswap kalith socket
Parts:
- removed MX14, MX15, MX63: 1u, MX_Only:MXOnly-1U-NoLED
- removed MX33, MX75: 1.25u, MX_Only:MXOnly-1.25U-NoLED
- removed MX62, MX64: 1.5u, MX_Only:MXOnly-1.5U-NoLED
- removed MX65: 7u, MX_Only:MXOnly-7U-ReversedStabilizers-NoLED
- MX1, MX10, MX11, MX12, MX13, MX16, MX19, MX2, MX20, MX21, MX22, MX23, MX24, MX25, MX26, MX27, MX28, MX29, MX3, MX30, MX32, MX35, MX36, MX37, MX38, MX39, MX4, MX40, MX41, MX42, MX43, MX44, MX45, MX47, MX49, MX5, MX50, MX51, MX52, MX53, MX54, MX55, MX56, MX57, MX58, MX6, MX60, MX61, MX68, MX69, MX7, MX70, MX8, MX9: footprint MX_Only:MXOnly-1U-NoLED -> Official_Switch_Keyboard_Hotswap_Kailh:SW_Hotswap_Kailh_MX_1.00u
- MX17: footprint MX_Only:MXOnly-2U-NoLED -> Official_Switch_Keyboard_Hotswap_Kailh:SW_Hotswap_Kailh_MX_2.00u
- MX18, MX31, MX67: footprint MX_Only:MXOnly-1.5U-NoLED -> Official_Switch_Keyboard_Hotswap_Kailh:SW_Hotswap_Kailh_MX_1.50u
- MX34, MX59: footprint MX_Only:MXOnly-1.75U-NoLED -> Official_Switch_Keyboard_Hotswap_Kailh:SW_Hotswap_Kailh_MX_1.75u
- MX46, MX48: footprint MX_Only:MXOnly-2.25U-NoLED -> Official_Switch_Keyboard_Hotswap_Kailh:SW_Hotswap_Kailh_MX_2.25u
- MX66, MX71, MX72, MX73: footprint MX_Only:MXOnly-1.25U-NoLED -> Official_Switch_Keyboard_Hotswap_Kailh:SW_Hotswap_Kailh_MX_1.25u
- MX74: footprint MX_Only:MXOnly-6.25U-ReversedStabilizers-NoLED -> Official_Switch_Keyboard_Hotswap_Kailh:SW_Hotswap_Kailh_MX_6.25u
- moved R4 4.83 mm to (30.6, 51.2), turned to 180 degrees
- moved D32 4.14 mm to (26.6, 51.2), turned to 270 degrees
- moved U2 2.95 mm to (25.6, 37.8)
- moved C5 2.83 mm to (39.0, 32.9)
- moved C6 2.83 mm to (39.0, 38.5)
- moved Y1 2.83 mm to (39.0, 35.7)
- moved C2 2.62 mm to (14.6, 38.6)
- moved C1 2.50 mm to (34.7, 33.9)
- moved C3 2.46 mm to (29.6, 46.9)
- moved D68 1.69 mm to (285.2, 87.7)
- moved C7 1.52 mm to (26.6, 27.5)
- moved D60 1.50 mm to (21.7, 87.5)
- moved D61 1.50 mm to (25.7, 87.5)
- moved D66 1.50 mm to (264.6, 87.5)
- moved D67 1.50 mm to (267.8, 87.5)
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Connections:
- U1 pad 3: Net-(U1-Pad3) -> (no net)
- U1 pad 4: Net-(U1-Pad4) -> (no net)
- U2 pad 41: Net-(U2-Pad41) -> (no net)
- U2 pad 42: Net-(U2-Pad42) -> (no net)
Routing:
- net COL15: track 355.0 -> 0.00 mm
- net COL13: track 353.1 -> 0.00 mm
- net ROW4: track 346.6 -> 0.00 mm, vias 2 -> 0
- net COL14: track 318.9 -> 0.00 mm, vias 1 -> 0
- net COL12: track 318.3 -> 0.00 mm
- net ROW2: track 301.5 -> 0.00 mm, vias 2 -> 0
- net ROW3: track 300.9 -> 0.00 mm, vias 2 -> 0
- net ROW0: track 295.7 -> 0.00 mm, vias 2 -> 0
- net COL11: track 293.6 -> 0.00 mm
- net ROW1: track 284.9 -> 0.00 mm, vias 2 -> 0
- net COL9: track 266.7 -> 0.00 mm
- net COL10: track 254.7 -> 0.00 mm
- net COL8: track 217.4 -> 0.00 mm
- net COL6: track 212.1 -> 0.00 mm
- net COL7: track 198.8 -> 0.00 mm
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Other:
- net class D: trace_width 0.2 -> 0.35
- net class Default: trace_width 0.25 -> 0.45
- net class Power: trace_width 0.381 -> 0.4
