File: pcb/bakeneko-65-pcb.sch (KiCad schematic (older format))
At the start: 18 parts, among them J1 JST SH 4-pin, J2 AVR-ISP-6, SW1 Reset, U1 SRV05-4, U2 ATmega32U4-AU, Y1 16MHz

Commit message: Modified PCB for hotswap kalith socket
Parts:
- J2: symbol Connector:AVR-ISP-6 -> bakeneko-65-pcb-rescue:AVR-ISP-6-Connector
- U2: symbol MCU_Microchip_ATmega:ATmega32U4-AU -> bakeneko-65-pcb-rescue:ATmega32U4-AU-MCU_Microchip_ATmega
Changed lines of the file:
@@
 EESchema Schematic File Version 4
-LIBS:bakeneko-65-pcb-cache
 EELAYER 30 0
 EELAYER END
@@
 D+
 $Comp
-L MCU_Microchip_ATmega:ATmega32U4-AU U2
+L bakeneko-65-pcb-rescue:ATmega32U4-AU-MCU_Microchip_ATmega U2
 U 1 1 5F26004F
 P 2300 5050
@@
 	5350 5150 5650 5150
 $Comp
-L Connector:AVR-ISP-6 J2
+L bakeneko-65-pcb-rescue:AVR-ISP-6-Connector J2
 U 1 1 5F4C9CCE
 P 2050 1700
