File: pcb/matrix.sch (KiCad schematic (older format))
At the start: 143 parts

Commit message: Modified PCB for hotswap kalith socket
Parts:
- MX1, MX10, MX11, MX12, MX13, MX14, MX15, MX16, MX19, MX2, MX20, MX21, MX22, MX23, MX24, MX25, MX26, MX27, MX28, MX29, MX3, MX30, MX32, MX35, MX36, MX37, MX38, MX39, MX4, MX40, MX41, MX42, MX43, MX44, MX45, MX47, MX49, MX5, MX50, MX51, MX52, MX53, MX54, MX55, MX56, MX57, MX58, MX6, MX60, MX61, MX63, MX68, MX69, MX7, MX70, MX8, MX9: footprint MX_Only:MXOnly-1U-NoLED -> Official_Switch_Keyboard_Hotswap_Kailh:SW_Hotswap_Kailh_MX_1.00u
- MX17: footprint MX_Only:MXOnly-2U-NoLED -> Official_Switch_Keyboard_Hotswap_Kailh:SW_Hotswap_Kailh_MX_2.00u
- MX18, MX31, MX62, MX64, MX67: footprint MX_Only:MXOnly-1.5U-NoLED -> Official_Switch_Keyboard_Hotswap_Kailh:SW_Hotswap_Kailh_MX_1.50u
- MX33, MX66, MX71, MX72, MX73, MX75: footprint MX_Only:MXOnly-1.25U-NoLED -> Official_Switch_Keyboard_Hotswap_Kailh:SW_Hotswap_Kailh_MX_1.25u
- MX34, MX59: footprint MX_Only:MXOnly-1.75U-NoLED -> Official_Switch_Keyboard_Hotswap_Kailh:SW_Hotswap_Kailh_MX_1.75u
- MX46, MX48: footprint MX_Only:MXOnly-2.25U-NoLED -> Official_Switch_Keyboard_Hotswap_Kailh:SW_Hotswap_Kailh_MX_2.25u
- MX65: footprint MX_Only:MXOnly-7U-ReversedStabilizers-NoLED -> Official_Switch_Keyboard_Hotswap_Kailh:SW_Hotswap_Kailh_MX_7.00u
- MX74: footprint MX_Only:MXOnly-6.25U-ReversedStabilizers-NoLED -> Official_Switch_Keyboard_Hotswap_Kailh:SW_Hotswap_Kailh_MX_6.25u
